File: pcbs/isolator/Isolator.kicad_pcb (KiCad board)
At the start: 2 copper layers, 30.5 x 17.8 mm, 11 parts, among them J1 USB-to-UART, J2 Power, J3 UART-to-Device, J4 Power, U1 FOD8012

Commit message: Updated PCBs
Routing:
- added copper zone on B.Cu, net GND
- added copper zone on F.Cu, net GND
- added copper zone on B.Cu, net GNDA
- added copper zone on F.Cu, net GNDA
Changed lines of the file:
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@@
     (links 22)
     (no_connects 0)
-    (area 0 0 0 0)
+    (area 116.764999 96.444999 147.395001 114.375001)
     (thickness 1.6)
     (drawings 5)
@@
       )
     )
+  )
+  (zone (net 5) (net_name GND) (layer F.Cu) (hatch edge 0.508)
+    (connect_pads (clearance 0.508))
+    (min_thickness 0.254)
+    (fill yes (arc_segments 16) (thermal_gap 0.508) (thermal_bridge_width 0.508))
+    (polygon
+      (pts
+        (xy 117.475 97.155) (xy 130.175 97.155) (xy 130.175 113.665) (xy 117.475 113.665)
+      )
+    )
+  )
+  (zone (net 5) (net_name GND) (layer B.Cu) (hatch edge 0.508)
+    (connect_pads (clearance 0.508))
+    (min_thickness 0.254)
+    (fill yes (arc_segments 16) (thermal_gap 0.508) (thermal_bridge_width 0.508))
+    (polygon
+      (pts
+        (xy 117.475 97.155) (xy 130.175 97.155) (xy 130.175 113.665) (xy 117.475 113.665)
+      )
+    )
+  )
+  (zone (net 4) (net_name GNDA) (layer F.Cu) (hatch edge 0.508)
+    (connect_pads (clearance 0.508))
+    (min_thickness 0.254)
+    (fill yes (arc_segments 16) (thermal_gap 0.508) (thermal_bridge_width 0.508))
+    (polygon
+      (pts
+        (xy 133.985 97.155) (xy 146.685 97.155) (xy 146.685 113.665) (xy 133.985 113.665)
+      )
+    )
+  )
+  (zone (net 4) (net_name GNDA) (layer B.Cu) (hatch edge 0.508)
+    (connect_pads (clearance 0.508))
+    (min_thickness 0.254)
+    (fill yes (arc_segments 16) (thermal_gap 0.508) (thermal_bridge_width 0.508))
+    (polygon
+      (pts
+        (xy 133.985 97.155) (xy 146.685 97.155) (xy 146.685 113.665) (xy 133.985 113.665)
+      )
+    )
