File: pcbs/devboard/Devboard.sch (KiCad schematic (older format))
At the start: 11 parts, among them J1 Power, J2 Left, J3 ARM-JTAG, J4 Right, J5 JTAG, SW1 SW_Push, U1 Trådfri

Commit message: Updated devboard pcb, accidentally swapped GND and VCC line.
Changed lines of the file:
@@
 LIBS:switches
 LIBS:jtag10
+LIBS:Devboard-cache
 EELAYER 25 0
 EELAYER END
@@
 L GND #PWR01
 U 1 1 5A0E1FA1
-P 2550 1900
-F 0 "#PWR01" H 2550 1650 50  0001 C CNN
-F 1 "GND" H 2550 1750 50  0000 C CNN
-F 2 "" H 2550 1900 50  0001 C CNN
-F 3 "" H 2550 1900 50  0001 C CNN
-	1    2550 1900
+P 2550 2050
+F 0 "#PWR01" H 2550 1800 50  0001 C CNN
+F 1 "GND" H 2550 1900 50  0000 C CNN
+F 2 "" H 2550 2050 50  0001 C CNN
+F 3 "" H 2550 2050 50  0001 C CNN
+	1    2550 2050
 	1    0    0    -1
 $EndComp
@@
 L +3V3 #PWR02
 U 1 1 5A0E1FC1
-P 2550 1150
-F 0 "#PWR02" H 2550 1000 50  0001 C CNN
-F 1 "+3V3" H 2550 1290 50  0000 C CNN
-F 2 "" H 2550 1150 50  0001 C CNN
-F 3 "" H 2550 1150 50  0001 C CNN
-	1    2550 1150
+P 2650 950
+F 0 "#PWR02" H 2650 800 50  0001 C CNN
+F 1 "+3V3" H 2650 1090 50  0000 C CNN
+F 2 "" H 2650 950 50  0001 C CNN
+F 3 "" H 2650 950 50  0001 C CNN
+	1    2650 950
 	1    0    0    -1
 $EndComp
@@
 Text Label 4800 1050 0    60   ~ 0
 RESETn
-Text Label 3300 2400 3    60   ~ 0
+Text Label 3300 2500 3    60   ~ 0
 RESETn
 $Comp
@@
 Text Label 6500 3250 2    60   ~ 0
 SWO
+Text Notes 3650 750  0    60   ~ 12
+UNTESTED
 Wire Wire Line
 	6050 3250 6500 3250
@@
 	3300 3250 3300 3450
 Wire Wire Line
-	3300 2400 3300 2850
-Connection ~ 2550 1750
-Wire Wire Line
-	2550 1750 2550 1900
+	3300 2500 3300 2850
+Wire Wire Line
+	4450 1950 5450 1950
+Wire Wire Line
+	4450 1850 5450 1850
+Wire Wire Line
+	4450 1750 5450 1750
+Wire Wire Line
+	4450 1650 5450 1650
+Wire Wire Line
+	4450 1550 5450 1550
+Wire Wire Line
+	4450 1450 5450 1450
+Wire Wire Line
+	4450 1350 5450 1350
+Wire Wire Line
+	4450 1250 5450 1250
+Wire Wire Line
+	4450 1150 5450 1150
+Wire Wire Line
+	4450 1050 5450 1050
+Wire Wire Line
+	2450 1750 3450 1750
+Wire Wire Line
+	2450 1650 3450 1650
+Wire Wire Line
+	2450 1550 3450 1550
+Wire Wire Line
+	2450 1450 3450 1450
+Wire Wire Line
+	2450 1350 3450 1350
+Wire Wire Line
+	2450 1250 3450 1250
+Wire Wire Line
+	2650 950  2650 1750
+Connection ~ 2650 1750
+Wire Wire Line
+	2550 1650 2550 2050
 Connection ~ 2550 1650
-Wire Wire Line
-	2550 1650 2550 1150
-Wire Wire Line
-	4450 1950 5450 1950
-Wire Wire Line
-	4450 1850 5450 1850
-Wire Wire Line
-	4450 1750 5450 1750
-Wire Wire Line
-	4450 1650 5450 1650
-Wire Wire Line
-	4450 1550 5450 1550
-Wire Wire Line
-	4450 1450 5450 1450
-Wire Wire Line
-	4450 1350 5450 1350
-Wire Wire Line
-	4450 1250 5450 1250
-Wire Wire Line
-	4450 1150 5450 1150
-Wire Wire Line
-	4450 1050 5450 1050
-Wire Wire Line
-	2450 1750 3450 1750
-Wire Wire Line
-	2450 1650 3450 1650
-Wire Wire Line
-	2450 1550 3450 1550
-Wire Wire Line
-	2450 1450 3450 1450
-Wire Wire Line
-	2450 1350 3450 1350
-Wire Wire Line
-	2450 1250 3450 1250
-Text Notes 3650 750  0    60   ~ 12
-UNTESTED
 $EndSCHEMATC

Commit message: Updated PCBs
Parts:
- removed U1: Trådfri, Parts:Trådfri PCB2.0, symbol Trådfri
- added U1: TRADFRI, IKEA:TRADFRI_PCB2.0, symbol TRADFRI
Changed lines of the file:
@@
 LIBS:contrib
 LIBS:valves
-LIBS:trådfri
+LIBS:ikea
 LIBS:switches
-LIBS:jtag10
-LIBS:Devboard-cache
 EELAYER 25 0
 EELAYER END
@@
 Comment4 ""
 $EndDescr
-$Comp
-L Trådfri U1
-U 1 1 5A0E1C08
-P 4150 1250
-F 0 "U1" H 3650 1600 60  0000 C CNN
-F 1 "Trådfri" H 4150 1600 60  0000 C CNN
-F 2 "Parts:Trådfri PCB2.0" H 4150 1250 60  0001 C CNN
-F 3 "" H 4150 1250 60  0001 C CNN
-	1    4150 1250
-	1    0    0    -1
-$EndComp
 $Comp
 L Conn_01x10 J4
@@
 	2550 1650 2550 2050
 Connection ~ 2550 1650
+$Comp
+L TRADFRI U1
+U 1 1 5A1186AF
+P 4150 1250
+F 0 "U1" H 3650 1600 60  0000 C CNN
+F 1 "TRADFRI" H 4150 1600 60  0000 C CNN
+F 2 "IKEA:TRADFRI_PCB2.0" H 4150 1250 60  0001 C CNN
+F 3 "" H 4150 1250 60  0001 C CNN
+	1    4150 1250
+	1    0    0    -1
+$EndComp
 $EndSCHEMATC

Commit message: Fixed edge cuts. Upgrade tot Kicad 5.0-rc2.
Parts:
- C1: symbol CP -> Devboard-rescue:CP
- C2: symbol C -> Devboard-rescue:C
- D1: symbol LED -> Devboard-rescue:LED
- J1: symbol Conn_01x02 -> Devboard-rescue:Conn_01x02
- J2: symbol Conn_01x06 -> Devboard-rescue:Conn_01x06
- J3: symbol Conn_02x05_Odd_Even -> Devboard-rescue:Conn_02x05_Odd_Even
- J4: symbol Conn_01x10 -> Devboard-rescue:Conn_01x10
- J5: symbol Conn_02x03_Odd_Even -> Devboard-rescue:Conn_02x03_Odd_Even
- R1: symbol R -> Devboard-rescue:R
- SW1: value SW_Push -> RESET; symbol SW_Push -> Devboard-rescue:SW_Push
- U1: symbol TRADFRI -> Devboard-rescue:TRADFRI
Changed lines of the file:
@@
-EESchema Schematic File Version 2
-LIBS:power
-LIBS:device
-LIBS:transistors
-LIBS:conn
-LIBS:linear
-LIBS:regul
-LIBS:74xx
-LIBS:cmos4000
-LIBS:adc-dac
-LIBS:memory
-LIBS:xilinx
-LIBS:microcontrollers
-LIBS:dsp
-LIBS:microchip
-LIBS:analog_switches
-LIBS:motorola
-LIBS:texas
-LIBS:intel
-LIBS:audio
-LIBS:interface
-LIBS:digital-audio
-LIBS:philips
-LIBS:display
-LIBS:cypress
-LIBS:siliconi
-LIBS:opto
-LIBS:atmel
-LIBS:contrib
-LIBS:valves
-LIBS:ikea
-LIBS:switches
-EELAYER 25 0
+EESchema Schematic File Version 4
+LIBS:Devboard-cache
+EELAYER 26 0
 EELAYER END
 $Descr User 8268 5827
@@
 $EndDescr
 $Comp
-L Conn_01x10 J4
+L Devboard-rescue:Conn_01x10 J4
 U 1 1 5A0E1C62
 P 5650 1450
@@
 $EndComp
 $Comp
-L Conn_01x06 J2
+L Devboard-rescue:Conn_01x06 J2
 U 1 1 5A0E1D8E
 P 2250 1450
@@
 $EndComp
 $Comp
-L GND #PWR01
+L Devboard-rescue:GND #PWR01
 U 1 1 5A0E1FA1
 P 2550 2050
@@
 $EndComp
 $Comp
-L +3V3 #PWR02
+L Devboard-rescue:+3V3 #PWR02
 U 1 1 5A0E1FC1
 P 2650 950
@@
 $EndComp
 $Comp
-L SW_Push SW1
+L Devboard-rescue:SW_Push SW1
 U 1 1 5A0E2005
 P 3300 3050
 F 0 "SW1" H 3350 3150 50  0000 L CNN
-F 1 "SW_Push" H 3300 2990 50  0000 C CNN
+F 1 "RESET" H 3300 2990 50  0000 C CNN
 F 2 "Buttons_Switches_THT:SW_PUSH_6mm" H 3300 3250 50  0001 C CNN
 F 3 "" H 3300 3250 50  0001 C CNN
@@
 $EndComp
 $Comp
-L GND #PWR03
+L Devboard-rescue:GND #PWR03
 U 1 1 5A0E2092
 P 3300 3450
@@
 $EndComp
 $Comp
-L Conn_01x02 J1
+L Devboard-rescue:Conn_01x02 J1
 U 1 1 5A0E2151
 P 1650 3050
@@
 $EndComp
 $Comp
-L GND #PWR04
+L Devboard-rescue:GND #PWR04
 U 1 1 5A0E2249
 P 5300 2100
@@
 $EndComp
 $Comp
-L GND #PWR05
+L Devboard-rescue:GND #PWR05
 U 1 1 5A0E22BF
 P 2000 3150
@@
 $EndComp
 $Comp
-L +3V3 #PWR06
+L Devboard-rescue:+3V3 #PWR06
 U 1 1 5A0E22D9
 P 2000 2850
@@
 $EndComp
 $Comp
-L +3V3 #PWR07
+L Devboard-rescue:+3V3 #PWR07
 U 1 1 5A0E237F
 P 2350 2600
@@
 $EndComp
 $Comp
-L LED D1
+L Devboard-rescue:LED D1
 U 1 1 5A0E23A0
 P 2350 2850
@@
 $EndComp
 $Comp
-L R R1
+L Devboard-rescue:R R1
 U 1 1 5A0E24CE
 P 2350 3200
@@
 $EndComp
 $Comp
-L GND #PWR08
+L Devboard-rescue:GND #PWR08
 U 1 1 5A0E251C
 P 2350 3450
@@
 $EndComp
 $Comp
-L CP C1
+L Devboard-rescue:CP C1
 U 1 1 5A0E2BAB
 P 2700 3000
@@
 $EndComp
 $Comp
-L C C2
+L Devboard-rescue:C C2
 U 1 1 5A0E2C05
 P 3000 3000
@@
 $EndComp
 $Comp
-L +3V3 #PWR09
+L Devboard-rescue:+3V3 #PWR09
 U 1 1 5A0E2C4D
 P 2700 2600
@@
 $EndComp
 $Comp
-L +3V3 #PWR010
+L Devboard-rescue:+3V3 #PWR010
 U 1 1 5A0E2C73
 P 3000 2600
@@
 $EndComp
 $Comp
-L GND #PWR011
+L Devboard-rescue:GND #PWR011
 U 1 1 5A0E2C99
 P 2700 3450
@@
 $EndComp
 $Comp
-L GND #PWR012
+L Devboard-rescue:GND #PWR012
 U 1 1 5A0E2CBF
 P 3000 3450
@@
 $EndComp
 $Comp
-L Conn_02x05_Odd_Even J3
+L Devboard-rescue:Conn_02x05_Odd_Even J3
 U 1 1 5A0E3330
 P 4200 3150
@@
 $EndComp
 $Comp
-L Conn_02x03_Odd_Even J5
+L Devboard-rescue:Conn_02x03_Odd_Even J5
 U 1 1 5A0E338C
 P 5750 3150
@@
 NoConn ~ 4500 3250
 $Comp
-L GND #PWR013
+L Devboard-rescue:GND #PWR013
 U 1 1 5A0E39B3
 P 3800 3450
@@
 $EndComp
 $Comp
-L +3V3 #PWR014
+L Devboard-rescue:+3V3 #PWR014
 U 1 1 5A0E3B30
 P 3800 2600
@@
 RESETn
 $Comp
-L +3V3 #PWR015
+L Devboard-rescue:+3V3 #PWR015
 U 1 1 5A0E44AE
 P 5150 2600
@@
 $EndComp
 $Comp
-L GND #PWR016
+L Devboard-rescue:GND #PWR016
 U 1 1 5A0E44DA
 P 5150 3450
@@
 Wire Wire Line
 	3800 3350 4000 3350
-Connection ~ 3800 3050
-Wire Wire Line
-	3800 3050 3800 3450
+Wire Wire Line
+	3800 3050 3800 3150
 Wire Wire Line
 	3800 3150 4000 3150
@@
 	3300 2500 3300 2850
 Wire Wire Line
-	4450 1950 5450 1950
+	4450 1950 5300 1950
 Wire Wire Line
 	4450 1850 5450 1850
@@
 	4450 1050 5450 1050
 Wire Wire Line
-	2450 1750 3450 1750
-Wire Wire Line
-	2450 1650 3450 1650
+	2450 1750 2650 1750
+Wire Wire Line
+	2450 1650 2550 1650
 Wire Wire Line
 	2450 1550 3450 1550
@@
 Connection ~ 2550 1650
 $Comp
-L TRADFRI U1
+L Devboard-rescue:TRADFRI U1
 U 1 1 5A1186AF
 P 4150 1250
@@
 	1    0    0    -1
 $EndComp
+Wire Wire Line
+	3800 3350 3800 3450
+Wire Wire Line
+	3800 3150 3800 3350
+Wire Wire Line
+	5300 1950 5450 1950
+Wire Wire Line
+	2650 1750 3450 1750
+Wire Wire Line
+	2550 1650 3450 1650
 $EndSCHEMATC
